File: pcb/sensorinterface/sensorinterface.kicad_sch (KiCad schematic)
At the start: 15 parts, among them J1 Conn_01x03, J2 Conn_01x03, J3 Conn_01x05, U1 LM393

Commit message: Add LEDs.
Parts:
- added C4: C, Capacitor_SMD:C_0603_1608Metric, symbol Device:C
- added D1, D2: LED, LED_SMD:LED_0603_1608Metric, symbol Device:LED
- added R7, R8: 1k, Resistor_SMD:R_0603_1608Metric, symbol Device:R
- R1, R2: value 1k -> 680
Connections:
- net +3.3V: now also C4.1
- net GND: now also C4.2, D1.1 (K), D2.1 (K)
- net at J3.3 (Pin_3), R1.2, U1.1: now also R8.1
- net at J3.4 (Pin_4), R2.2, U1.7: now also R7.1
- new net: D2.2 (A), R7.2
- new net: D1.2 (A), R8.2
Other:
- note added: "+3.3V"
- note added: "+5V"
- note added: "GND"
- note added: "OUT1"
- note added: "OUT2"

Commit message: Complete routing.
Parts:
- R3, R4, R5, R6: value R -> 2k
- RV1, RV2: value 10k -> 1k; footprint (none) -> Potentiometer_THT:Potentiometer_Trimmer_ACP_CA6v_Horizontal
Changed lines of the file:
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@@
 			)
 		)
-		(property "Value" "10k"
-			(at 35.56 32.385 90)
+		(property "Value" "1k"
+			(at 35.56 33.02 90)
 			(show_name no)
 			(do_not_autoplace no)
@@
 			)
 		)
-		(property "Footprint" ""
+		(property "Footprint" "Potentiometer_THT:Potentiometer_Trimmer_ACP_CA6v_Horizontal"
 			(at 35.56 34.29 0)
 			(hide yes)
@@
 		(in_pos_files yes)
 		(dnp no)
-		(fields_autoplaced yes)
 		(property "Reference" "R5"
 			(at 38.1 76.1999 0)
@@
 			)
 		)
-		(property "Value" "R"
-			(at 38.1 78.7399 0)
+		(property "Value" "2k"
+			(at 35.56 78.74 90)
 			(show_name no)
 			(do_not_autoplace no)
@@
 		(in_pos_files yes)
 		(dnp no)
-		(fields_autoplaced yes)
 		(property "Reference" "R4"
 			(at 38.1 24.1299 0)
@@
 			)
 		)
-		(property "Value" "R"
-			(at 38.1 26.6699 0)
+		(property "Value" "2k"
+			(at 35.56 26.67 90)
 			(show_name no)
 			(do_not_autoplace no)
@@
 		(in_pos_files yes)
 		(dnp no)
-		(fields_autoplaced yes)
 		(property "Reference" "R3"
 			(at 38.1 41.9099 0)
@@
 			)
 		)
-		(property "Value" "R"
-			(at 38.1 44.4499 0)
+		(property "Value" "2k"
+			(at 35.56 44.45 90)
 			(show_name no)
 			(do_not_autoplace no)
@@
 			)
 		)
-		(property "Value" "10k"
-			(at 35.56 84.455 90)
+		(property "Value" "1k"
+			(at 35.56 85.09 90)
 			(show_name no)
 			(do_not_autoplace no)
@@
 			)
 		)
-		(property "Footprint" ""
+		(property "Footprint" "Potentiometer_THT:Potentiometer_Trimmer_ACP_CA6v_Horizontal"
 			(at 35.56 86.36 0)
 			(hide yes)
@@
 		(in_pos_files yes)
 		(dnp no)
-		(fields_autoplaced yes)
 		(property "Reference" "R6"
 			(at 38.1 93.9799 0)
@@
 			)
 		)
-		(property "Value" "R"
-			(at 38.1 96.5199 0)
-			(show_name no)
-			(do_not_autoplace no)
+		(property "Value" "2k"
+			(at 35.56 96.52 90)
+			(show_name no)
+			(do_not_autoplace no)
